File: PCB.kicad_pcb (KiCad board)
At the start: 2 copper layers, 112.5 x 136.1 mm, 73 parts, among them J1 USB_C_Receptacle_USB2.0_16P, J10 Conn_01x03_Pin, J2 Conn_01x03_Pin, J3 USB_C_Receptacle_USB2.0_16P, J4 Conn_01x08_Socket, J5 Conn_01x02_Pin, J6 Conn_01x04_Pin, J7 Conn_01x07_Pin, J9 Conn_01x03_Pin, Q1 S8050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

Commit message: debut rootage
Parts:
- removed the H1 at (231.5, 106.2)
- removed the H2 at (267.5, 100.2)
- removed the H3 at (237.5, 142.2)
- removed the H4 at (273.5, 136.2)
- Q1, Q2: footprint Package_TO_SOT_THT:TO-92_Inline -> Package_TO_SOT_SMD:SOT-23-3
- moved R10 172.5 mm to (187.0, 135.1), turned to -90 degrees
- moved R6 163.5 mm to (187.5, 82.2), turned to -90 degrees
- moved R5 161.1 mm to (185.0, 82.2), turned to -90 degrees
- moved C9 160.3 mm to (189.2, 128.0), turned to -90 degrees
- moved I2C1 157.5 mm to (185.8, 93.0), turned to 90 degrees
- moved C2 155.5 mm to (184.0, 135.0), turned to -90 degrees
- moved C10 149.8 mm to (185.8, 128.6), turned to -90 degrees
- moved C11 145.8 mm to (182.8, 128.6), turned to -90 degrees
- moved R1 145.1 mm to (149.8, 134.4), turned to 90 degrees
- moved SW2 143.7 mm to (180.5, 134.5), turned to 90 degrees
- moved C17 139.7 mm to (172.8, 114.4), turned to 180 degrees
- moved C19 137.5 mm to (179.8, 128.6), turned to -90 degrees
- moved Q1 135.6 mm to (146.3, 131.6)
- moved Q2 130.9 mm to (146.3, 127.6)
- moved J6 129.8 mm to (193.5, 88.3), turned to -90 degrees
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Connections:
- C14 pad 1: unconnected-(C14-Pad1) -> BTN1
- C15 pad 1: unconnected-(C15-Pad1) -> BTN2
- C16 pad 1: unconnected-(C16-Pad1) -> BTN3
- Q2 pad 1: BOOT -> DTR
- Q2 pad 3: DTR -> BOOT
Routing:
- net GND: track 0.00 -> 85.4 mm, vias 0 -> 35
- net 3V3: track 0.00 -> 82.4 mm, vias 0 -> 7
- net SCL: track 0.00 -> 68.7 mm, vias 0 -> 2
- net SDA: track 0.00 -> 65.3 mm, vias 0 -> 2
- net NEOPIXEL: track 0.00 -> 58.3 mm, vias 0 -> 2
- net WS: track 0.00 -> 57.0 mm, vias 0 -> 2
- net SD_MIC: track 0.00 -> 53.3 mm, vias 0 -> 1
- net DC: track 0.00 -> 48.5 mm, vias 0 -> 2
- net ROTA: track 0.00 -> 47.1 mm, vias 0 -> 1
- net EN: track 0.00 -> 45.9 mm
- net VCC_5V: track 0.00 -> 44.1 mm
- net RX0: track 0.00 -> 42.6 mm, vias 0 -> 2
- net CLK: track 0.00 -> 42.5 mm, vias 0 -> 2
- net CS: track 0.00 -> 38.3 mm, vias 0 -> 4
- net ROTB: track 0.00 -> 38.2 mm, vias 0 -> 1
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- added copper zone on F.Cu, net 3V3
- added copper zone on B.Cu, net GND
- added copper zone on F.Cu, net VBUS_NP
- added copper zone on F.Cu, net VBUS_UART
- added copper zone on F.Cu, net VCC_5V
Other:
- board size 112.5 x 136.1 mm -> 60 x 60 mm

Commit message: fin routage
Parts:
- moved R1 2.32 mm to (147.6, 135.2), turned to 180 degrees
- moved R5 0.60 mm to (184.4, 82.2)
- moved R6 0.50 mm to (187.0, 82.2)
- moved JP1 0.36 mm to (165.9, 114.0), turned to 0 degrees
Connections:
- U6 pad 12: SD_MIC -> WS
- U6 pad 18: ROTA -> CLK
- U6 pad 19: ROTB -> MOSI
- U6 pad 20: ROTS1 -> SCLK
- U6 pad 21: MOSI -> CS
- U6 pad 22: SCLK -> DC
- U6 pad 24: CLK -> BLK
- U6 pad 25: BLK -> NEOPIXEL
- U6 pad 31: WS -> SD_MIC
- U6 pad 4: NEOPIXEL -> BTN1
- U6 pad 5: BTN1 -> BTN2
- U6 pad 6: BTN2 -> BTN3
- U6 pad 7: BTN3 -> ROTS1
- U6 pad 8: CS -> ROTA
- U6 pad 9: DC -> ROTB
Routing:
- net 3V3: track 82.4 -> 262.4 mm, vias 7 -> 1
- net VCC_5V: track 44.1 -> 125.6 mm, vias 0 -> 3
- net GND: track 85.4 -> 26.0 mm, vias 35 -> 154
- net BTN1: track 4.59 -> 58.2 mm, vias 1 -> 4
- net BTN2: track 5.52 -> 53.6 mm, vias 1 -> 4
- net BTN3: track 1.25 -> 47.0 mm, vias 1 -> 4
- net NEOPIXEL: track 58.3 -> 32.8 mm
- net CLK: track 42.5 -> 65.4 mm, vias 2 -> 1
- net DC: track 48.5 -> 28.8 mm, vias 2 -> 1
- net ROTB: track 38.2 -> 57.7 mm, vias 1 -> 3
- net WS: track 57.0 -> 75.9 mm
- net MOSI: track 21.1 -> 35.9 mm
- net ROTS1: track 30.5 -> 44.7 mm, vias 1 -> 3
- net ROTA: track 47.1 -> 61.0 mm, vias 1 -> 3
- net SD_MIC: track 53.3 -> 39.6 mm, vias 1 -> 2
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- added copper zone on F.Cu, net GND
- removed copper zone on F.Cu, net 3V3
- removed copper zone on F.Cu, net VCC_5V
Other:
- board text added: "+VOL"
- board text added: "3.3V"
- board text added: "3V3"
- board text added: "5V"
- board text added: "AMPLIFIER"
- board text added: "BOOT"
- board text added: "BTN1"
- board text added: "BTN2"
- board text added: "BTN3"
- board text added: "CLK WS GND SD 3V3 GND"
- board text added: "COM"
- board text added: "GND"
- board text added: "I2C"
- board text added: "MICRO"
- board text added: "NEOPIXEL"
- board text added: "RESET"
- board text added: "ROT ENCODER"
- board text added: "RX"
- board text added: "SCL"
- board text added: "SCREEN"
- board text added: "SDA"
- board text added: "TX"
- board text added: "UART1"
- board text added: "USB"

Commit message: test DRC
Parts:
- moved J4 17.9 mm to (157.0, 98.8), turned to 90 degrees
- moved J7 15.2 mm to (173.4, 110.8), turned to -90 degrees
- moved JP1 0.70 mm to (166.6, 114.0)
- moved C17 0.50 mm to (173.3, 114.4)
Connections:
- U6 pad 17: DIN -> CLK
- U6 pad 18: CLK -> DIN
- U6 pad 19: MOSI -> BLK
- U6 pad 20: SCLK -> RST
- U6 pad 21: CS -> DC
- U6 pad 22: DC -> CS
- U6 pad 23: RST -> SCLK
- U6 pad 24: BLK -> MOSI
Routing:
- net WS: track 75.9 -> 58.7 mm, vias 2 -> 6
- net 3V3: track 262.4 -> 277.7 mm, vias 1 -> 4
- net BLK: track 26.4 -> 39.9 mm
- net RST: track 27.5 -> 37.6 mm
- net CLK: track 65.4 -> 55.3 mm, vias 1 -> 3
- net MOSI: track 35.9 -> 29.2 mm
- net DC: track 28.8 -> 35.5 mm
- net DIN: track 12.5 -> 7.63 mm
- net VCC_5V: track 125.6 -> 128.6 mm
- net CS: track 30.5 -> 33.4 mm
- net SCLK: track 33.5 -> 31.8 mm
- net GND: track 26.0 -> 25.5 mm, vias 154 -> 156
- net (no net): vias 1 -> 0

Commit message: fin V1
Routing:
- net GND: vias 156 -> 196
Other:
- board text added: "TiToom 12/12/25 V1"

Commit message: update V2
Parts:
- removed C1: 100nF, Capacitor_SMD:C_0805_2012Metric_Pad1.18x1.45mm_HandSolder
- removed D2, D7: ~, LED_SMD:LED_0805_2012Metric_Pad1.15x1.40mm_HandSolder
- removed D3, D4, D5: SS34, Diode_SMD:D_SMA_Handsoldering
- removed J3: USB_C_Receptacle_USB2.0_16P, Connector_USB:USB_C_Receptacle_HRO_TYPE-C-31-M-12
- removed J5: Conn_01x02_Pin, Connector_PinHeader_2.54mm:PinHeader_1x02_P2.54mm_Vertical
- removed Q1, Q2: S8050, Package_TO_SOT_SMD:SOT-23-3
- removed R11, R12: 5.1k, Resistor_SMD:R_0805_2012Metric_Pad1.20x1.40mm_HandSolder
- removed R13, R14: 10k, Resistor_SMD:R_1206_3216Metric_Pad1.30x1.75mm_HandSolder
- removed R8, R9: 470, Resistor_SMD:R_0805_2012Metric_Pad1.20x1.40mm_HandSolder
- removed U1: CH340C, Package_SO:SOIC-16_3.9x9.9mm_P1.27mm
- removed U3: USBLC6-2SC6, Package_TO_SOT_SMD:SOT-23-6_Handsoldering
- added JP2: SolderJumper_2_Open, Jumper:SolderJumper-2_P1.3mm_Open_RoundedPad1.0x1.5mm, F.Cu at (182.1, 111.2)
- added JP3: SolderJumper_2_Open, Jumper:SolderJumper-2_P1.3mm_Open_RoundedPad1.0x1.5mm, F.Cu at (182.2, 105.2)
- moved R5 62.9 mm to (147.2, 132.9), turned to 0 degrees
- moved R6 62.0 mm to (147.2, 129.8), turned to 0 degrees
- moved J6 57.7 mm to (146.4, 121.6)
- moved I2C1 57.4 mm to (138.8, 125.9)
- moved UART1 54.5 mm to (138.8, 115.8), turned to 90 degrees
- moved D1 44.8 mm to (192.9, 122.4), turned to -90 degrees
- moved R4 43.0 mm to (192.8, 116.8)
- moved C12 21.8 mm to (144.2, 107.7), turned to 180 degrees
- moved SW3 13.8 mm to (184.7, 93.8), turned to 180 degrees
- moved D6 13.6 mm to (144.2, 103.4), turned to 180 degrees
- moved SW5 13.4 mm to (184.7, 81.8), turned to 180 degrees
- moved R7 12.8 mm to (150.6, 105.2)
- moved C14 9.66 mm to (177.8, 93.8), turned to 90 degrees
- moved C16 8.78 mm to (177.8, 81.8), turned to 90 degrees
- moved C8 6.66 mm to (169.6, 104.8)
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Connections:
- C14 pad 1: BTN1 -> BTN3
- C16 pad 1: BTN3 -> BTN1
- J1 pad A4: VBUS_NP -> VCC_5V
- J1 pad A9: VBUS_NP -> VCC_5V
- J1 pad B4: VBUS_NP -> VCC_5V
- J1 pad B9: VBUS_NP -> VCC_5V
- J6 pad 2: GND -> SDA
- J6 pad 3: SDA -> GND
- SW3 pad 2: BTN1 -> BTN3
- SW5 pad 2: BTN3 -> BTN1
- U2 pad 5: VBUS_NP -> VCC_5V
- U6 pad 10: TX1 -> MOSI
- U6 pad 11: RX1 -> NEOPIXEL
- U6 pad 24: MOSI -> unconnected-(U6-IO47-Pad24)
- U6 pad 25: NEOPIXEL -> unconnected-(U6-IO48-Pad25)
- U6 pad 38: SCL -> SDA
- U6 pad 39: SDA -> SCL
- UART1 pad 2: RX1 -> RX0
- UART1 pad 3: TX1 -> TX0
Routing:
- net 3V3: track 278.1 -> 203.7 mm, vias 4 -> 5
- net SCL: track 66.5 -> 27.6 mm
- net SDA: track 66.6 -> 30.6 mm, vias 1 -> 2
- net EN: track 45.2 -> 14.4 mm, vias 4 -> 2
- net USB_D+: track 23.2 -> 0.00 mm, vias 2 -> 0
- net USB_D-: track 21.9 -> 0.00 mm, vias 2 -> 0
- net TX1: track 19.7 -> 0.00 mm, vias 1 -> 0
- net RX1: track 19.6 -> 0.00 mm, vias 1 -> 0
- net VBUS_NP: track 18.6 -> 0.00 mm
- net Net-(D2-A): track 17.3 -> 0.00 mm, vias 2 -> 0
- net GND: track 25.5 -> 8.38 mm, vias 196 -> 262
- net VBUS_UART: track 16.8 -> 0.00 mm
- net MOSI: track 29.2 -> 44.4 mm
- net Net-(D7-A): track 14.8 -> 0.00 mm, vias 2 -> 0
- net Net-(J3-CC2): track 14.5 -> 0.00 mm, vias 2 -> 0
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- added copper zone on F.Cu, net VCC_5V
- removed copper zone on F.Cu, net VBUS_NP
- removed copper zone on F.Cu, net VBUS_UART
Other:
- board text added: "100n"
- board text added: "100u"
- board text added: "10k"
- board text added: "10n"
- board text added: "10u"
- board text added: "1u"
- board text added: "D_o"
- board text added: "RX0"
- board text added: "TX0"
- board text added: "TiToom 30/12/25 V2"
- board text added: "UART0"
- board text removed: "COM"
- board text removed: "RX"
- board text removed: "TX"
- board text removed: "TiToom 12/12/25 V1"
- board text removed: "UART1"
